File: Hardware/Attiny13A_Devboard_v1_SMD/Attiny13A_Devboard_v1_SMD.kicad_sch (KiCad schematic)
At the start: 0 parts

Commit message: Attiny13A Dev Board SMD - Finished Schematics
Signed-off-by: alexanderjg85 <alexanderjg85@gmail.com>
Parts:
- added C1: 10 uF, Capacitor_SMD:C_1206_3216Metric_Pad1.33x1.80mm_HandSolder, symbol Device:C_Small
- added C2: 100 nF, Capacitor_SMD:C_1206_3216Metric_Pad1.33x1.80mm_HandSolder, symbol Device:C_Small
- added D1: SS14, Diode_SMD:D_SMA_Handsoldering, symbol Diode:SS14
- added D2: RED, LED_SMD:LED_1206_3216Metric_Pad1.42x1.75mm_HandSolder, symbol Device:LED
- added J1: Screw_Terminal_01x02, TerminalBlock_Phoenix:TerminalBlock_Phoenix_MKDS-1,5-2-5.08_1x02_P5.08mm_Horizontal, symbol Connector:Screw_Terminal_01x02
- added J2: AVR-ISP-6, Connector_PinHeader_2.54mm:PinHeader_2x03_P2.54mm_Vertical, symbol Connector:AVR-ISP-6
- added J3: Conn_01x06_Pin, Connector_PinHeader_2.54mm:PinHeader_1x06_P2.54mm_Vertical, symbol Connector:Conn_01x06_Pin
- added R1: 470, Resistor_SMD:R_1206_3216Metric_Pad1.30x1.75mm_HandSolder, symbol Device:R_Small
- added R2: 10k, Resistor_SMD:R_1206_3216Metric_Pad1.30x1.75mm_HandSolder, symbol Device:R_Small
- added SW1: SW_Push, Button_Switch_SMD:SW_SPST_PTS647_Sx38, symbol Switch:SW_Push
- added U1: ATtiny13A-SS, Package_SO:SOIC-8_3.9x4.9mm_P1.27mm, symbol MCU_Microchip_ATtiny:ATtiny13A-SS
Connections:
- new net: D2.2 (A), R1.2
- new net +5V: D1.2 (A), J1.1 (Pin_1)
- new net AVR_LED: R1.1, U1.3 (PB4)
- new net AVR_MISO: J2.1 (MISO), J3.3 (Pin_3), U1.6 (PB1)
- new net AVR_MOSI: J2.4 (MOSI), J3.2 (Pin_2), U1.5 (PB0)
- new net AVR_PB3: J3.5 (Pin_5), U1.2 (PB3)
- new net AVR_RST: J2.5 (~{RST}), R2.2, SW1.1, U1.1 (~{RESET}/PB5)
- new net AVR_SCK: J2.3 (SCK), J3.4 (Pin_4), U1.7 (PB2)
- new net GND: C1.2, C2.1, D2.1 (K), J1.2 (Pin_2), J2.6 (GND), J3.6 (Pin_6), SW1.2, U1.4 (GND)
- new net VCC: C1.1, C2.2, D1.1 (K), J2.2 (VCC), J3.1 (Pin_1), R2.1, U1.8 (VCC)

Commit message: Attiny13A Dev Board SMD - Added Testpoints to Schematics
Signed-off-by: alexanderjg85 <alexanderjg85@gmail.com>
Parts:
- added TP1: TP_5V, TestPoint:TestPoint_Pad_D1.5mm, symbol Connector:TestPoint
- added TP2: TP_AVRLED, symbol Connector:TestPoint
- added TP3: TP_VCC, symbol Connector:TestPoint
- added TP4: TP_AVR_RST, symbol Connector:TestPoint
- added TP5: TP_AVR_PB3, symbol Connector:TestPoint
- added TP6: TP_AVR_SCK, symbol Connector:TestPoint
- added TP7: TP_AVR_MISO, symbol Connector:TestPoint
- added TP8: TP_AVR_MOSI, symbol Connector:TestPoint
Connections:
- net +5V: now also TP1.1
- net AVR_LED: now also TP2.1
- net AVR_MISO: now also TP7.1
- net AVR_MOSI: now also TP8.1
- net AVR_PB3: now also TP5.1
- net AVR_RST: now also TP4.1
- net AVR_SCK: now also TP6.1
- net VCC: now also TP3.1

Commit message: Attiny13A Dev Board SMD - Added Testpoints Footprint to Schematics
Signed-off-by: alexanderjg85 <alexanderjg85@gmail.com>
Parts:
- TP2, TP3, TP4, TP5, TP6, TP7, TP8: footprint (none) -> TestPoint:TestPoint_Pad_D1.5mm
Changed lines of the file:
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@@
 			)
 		)
-		(property "Footprint" ""
+		(property "Footprint" "TestPoint:TestPoint_Pad_D1.5mm"
 			(at 109.22 38.1 0)
 			(hide yes)
@@
 			)
 		)
-		(property "Footprint" ""
+		(property "Footprint" "TestPoint:TestPoint_Pad_D1.5mm"
 			(at 80.01 49.53 0)
 			(hide yes)
@@
 			)
 		)
-		(property "Footprint" ""
+		(property "Footprint" "TestPoint:TestPoint_Pad_D1.5mm"
 			(at 139.7 88.9 0)
 			(hide yes)
@@
 			)
 		)
-		(property "Footprint" ""
+		(property "Footprint" "TestPoint:TestPoint_Pad_D1.5mm"
 			(at 109.22 25.4 0)
 			(hide yes)
@@
 			)
 		)
-		(property "Footprint" ""
+		(property "Footprint" "TestPoint:TestPoint_Pad_D1.5mm"
 			(at 109.22 31.75 0)
 			(hide yes)
@@
 			)
 		)
-		(property "Footprint" ""
+		(property "Footprint" "TestPoint:TestPoint_Pad_D1.5mm"
 			(at 109.22 19.05 0)
 			(hide yes)
@@
 			)
 		)
-		(property "Footprint" ""
+		(property "Footprint" "TestPoint:TestPoint_Pad_D1.5mm"
 			(at 87.63 110.49 0)
 			(hide yes)

Commit message: Attiny13A Dev Board SMD - Layout - Initial Placement done
Signed-off-by: alexanderjg85 <alexanderjg85@gmail.com>
Parts:
- added TP9: TP_GND, TestPoint:TestPoint_Pad_D1.5mm, symbol Connector:TestPoint
Connections:
- net GND: now also TP9.1
Changed lines of the file:
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@@
+	)
+	(junction
+		(at 55.88 54.61)
+		(diameter 0)
+		(color 0 0 0 0)
 	)
 	(junction
@@
 	(wire
 		(pts
-			(xy 50.8 54.61) (xy 67.31 54.61)
+			(xy 50.8 54.61) (xy 55.88 54.61)
 		)
 		(stroke
@@
 		(pts
 			(xy 60.96 49.53) (xy 67.31 49.53)
+		)
+		(stroke
+			(width 0)
+			(type default)
+		)
+	)
+	(wire
+		(pts
+			(xy 55.88 54.61) (xy 67.31 54.61)
 		)
 		(stroke
@@
 					(unit 1)
 				)
+			)
+		)
+	)
+	(symbol
+		(lib_id "Connector:TestPoint")
+		(at 55.88 54.61 180)
+		(unit 1)
+		(body_style 1)
+		(exclude_from_sim no)
+		(in_bom yes)
+		(on_board yes)
+		(in_pos_files yes)
+		(dnp no)
+		(property "Reference" "TP9"
+			(at 57.15 59.944 0)
+			(show_name no)
+			(do_not_autoplace no)
+			(effects
+				(font
+					(size 1.27 1.27)
+				)
+				(justify left)
+			)
+		)
+		(property "Value" "TP_GND"
+			(at 64.516 57.15 0)
+			(show_name no)
+			(do_not_autoplace no)
+			(effects
+				(font
+					(size 1.27 1.27)
+				)
+				(justify left)
+			)
+		)
+		(property "Footprint" "TestPoint:TestPoint_Pad_D1.5mm"
+			(at 50.8 54.61 0)
+			(hide yes)
+			(show_name no)
+			(do_not_autoplace no)
+			(effects
+				(font
+					(size 1.27 1.27)
+				)
+			)
+		)
+		(property "Datasheet" ""
+			(at 50.8 54.61 0)
+			(hide yes)
+			(show_name no)
+			(do_not_autoplace no)
+			(effects
+				(font
+					(size 1.27 1.27)
+				)
+			)
+		)
+		(property "Description" "test point"
+			(at 55.88 54.61 0)
+			(hide yes)
+			(show_name no)
+			(do_not_autoplace no)
+			(effects
+				(font
+					(size 1.27 1.27)
+				)
+			)
+		)
+		(pin "1"
+		)
+		(instances
+			(project "Attiny13A_Devboard_v1_SMD"
+				(path "/5d112f69-b4bf-4615-b7c8-2f57c66ae4ee"
+					(reference "TP9")
+					(unit 1)
+				)

Commit message: Attiny13A Dev Board SMD - Layout - Optimized Silk Screen
Signed-off-by: alexanderjg85 <alexanderjg85@gmail.com>
Parts:
- J2: value AVR-ISP-6 -> ISP-6
- SW1: value SW_Push -> SW_RESET
- TP1: value TP_5V -> 5V
- TP2: value TP_AVRLED -> LED
- TP3: value TP_VCC -> VCC
- TP4: value TP_AVR_RST -> RST
- TP5: value TP_AVR_PB3 -> PB3
- TP6: value TP_AVR_SCK -> SCK
- TP7: value TP_AVR_MISO -> MISO
- TP8: value TP_AVR_MOSI -> MOSI
- TP9: value TP_GND -> GND
Changed lines of the file:
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@@
 			)
 		)
-		(property "Value" "TP_GND"
-			(at 64.516 57.15 0)
+		(property "Value" "GND"
+			(at 62.484 58.42 0)
 			(show_name no)
 			(do_not_autoplace no)
@@
 			)
 		)
-		(property "Value" "TP_5V"
-			(at 36.068 45.466 0)
+		(property "Value" "5V"
+			(at 38.354 45.72 0)
 			(show_name no)
 			(do_not_autoplace no)
@@
 			)
 		)
-		(property "Value" "TP_AVR_PB3"
-			(at 115.316 46.228 90)
+		(property "Value" "PB3"
+			(at 111.76 45.72 90)
 			(show_name no)
 			(do_not_autoplace no)
@@
 			)
 		)
-		(property "Value" "TP_VCC"
-			(at 66.294 46.99 0)
+		(property "Value" "VCC"
+			(at 69.342 46.228 0)
 			(show_name no)
 			(do_not_autoplace no)
@@
 			)
 		)
-		(property "Value" "TP_AVR_RST"
+		(property "Value" "RST"
 			(at 146.812 93.726 0)
 			(show_name no)
@@
 			)
 		)
-		(property "Value" "TP_AVR_MISO"
-			(at 115.316 33.528 90)
+		(property "Value" "MISO"
+			(at 112.522 33.528 90)
 			(show_name no)
 			(do_not_autoplace no)
@@
 			)
 		)
-		(property "Value" "TP_AVR_SCK"
-			(at 115.316 39.878 90)
+		(property "Value" "SCK"
+			(at 112.522 39.878 90)
 			(show_name no)
 			(do_not_autoplace no)
@@
 			)
 		)
-		(property "Value" "AVR-ISP-6"
+		(property "Value" "ISP-6"
 			(at 148.59 43.1799 0)
 			(show_name no)
@@
 			)
 		)
-		(property "Value" "TP_AVR_MOSI"
-			(at 115.316 27.178 90)
+		(property "Value" "MOSI"
+			(at 112.522 27.178 90)
 			(show_name no)
 			(do_not_autoplace no)
@@
 			)
 		)
-		(property "Value" "TP_AVRLED"
-			(at 71.374 108.204 0)
+		(property "Value" "LED"
+			(at 77.47 107.95 0)
 			(show_name no)
 			(do_not_autoplace no)
@@
 			)
 		)
-		(property "Value" "SW_Push"
+		(property "Value" "SW_RESET"
 			(at 189.738 93.218 0)
 			(show_name no)

Commit message: Attiny13A Dev Board SMD - Schematics - Added Part Properties
Signed-off-by: alexanderjg85 <alexanderjg85@gmail.com>
Parts:
- C1, C2: Package (none) -> 1206; Spec (none) -> 20% 16V
- D1: Package (none) -> SMA; Spec (none) -> 0.5A 30 V
- D2: Package (none) -> 1206; Spec (none) -> LED RED
- J1: Package (none) -> 5.08mm 1x2; Spec (none) -> Horizontal
- J2: Package (none) -> 2.54 mm 1x3; Spec (none) -> Male / THT/ Vertical
- J3: Package (none) -> 2.54 mm 1x6; Spec (none) -> Male / THT/ Vertical
- R1, R2: Package (none) -> 1206; Spec (none) -> 1% 125 mW
- SW1: Package (none) -> 4.5 x 4.5 SMD; Spec (none) -> H=5.0mm Tactile
- TP1, TP2, TP3, TP4, TP5, TP6, TP7, TP8, TP9: now left out of the parts list
- U1: MFR PN (none) -> ATTINY13A-SSU; Package (none) -> SOIC-8; Spec (none) -> 8-Bit AVR 20 Mhz

Commit message: Attiny13A Dev Board SMD - Updated Reset Switch Footprint for better Handsoldering - Optimized Silk Screen
Signed-off-by: alexanderjg85 <alexanderjg85@gmail.com>
Parts:
- SW1: footprint Button_Switch_SMD:SW_SPST_PTS647_Sx38 -> AJ_Electromechanical:SW_SPST_PTS647_Sx38_Handsolder; MFR PN (none) -> SWT0210-045026GSA; Spec H=5.0mm Tactile -> H=4.5mm Tactile
Changed lines of the file:
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@@
 			)
 		)
-		(property "Footprint" "Button_Switch_SMD:SW_SPST_PTS647_Sx38"
+		(property "Footprint" "AJ_Electromechanical:SW_SPST_PTS647_Sx38_Handsolder"
 			(at 190.5 86.36 0)
 			(hide yes)
@@
 			)
 		)
-		(property "Spec" "H=5.0mm Tactile"
+		(property "Spec" "H=4.5mm Tactile"
 			(at 190.5 91.44 0)
 			(hide yes)
+			(show_name no)
+			(do_not_autoplace no)
+			(effects
+				(font
+					(size 1.27 1.27)
+				)
+			)
+		)
+		(property "MFR PN" "SWT0210-045026GSA"
+			(at 190.5 91.44 0)
+			(hide yes)
